Commit message: Switch ur10 simulation to ros_controllers as well.

File: ur_description/urdf/ur.transmission.xacro (robot description, xacro)
@@ -4,5 +4,5 @@
        xmlns:interface="http://playerstage.sourceforge.net/gazebo/xmlschema/#interface"
        xmlns:xacro="http://ros.org/wiki/xacro">
-	<xacro:macro name="ur5_arm_transmission" params="name">
+	<xacro:macro name="ur_arm_transmission" params="prefix">
 		<transmission name="shoulder_pan_trans">
 			<type>transmission_interface/SimpleTransmission</type>
@@ -11,5 +11,5 @@
 				<mechanicalReduction>1</mechanicalReduction>
 			</actuator>
-			<joint name="${name}shoulder_pan_joint"/>
+			<joint name="${prefix}shoulder_pan_joint"/>
 		</transmission>
 		<transmission name="shoulder_lift_trans">
@@ -19,5 +19,5 @@
 				<mechanicalReduction>1</mechanicalReduction>
 			</actuator>
-			<joint name="${name}shoulder_lift_joint"/>
+			<joint name="${prefix}shoulder_lift_joint"/>
 		</transmission>
 		<transmission name="elbow_trans">
@@ -27,5 +27,5 @@
 				<mechanicalReduction>1</mechanicalReduction>
 			</actuator>
-			<joint name="${name}elbow_joint"/>
+			<joint name="${prefix}elbow_joint"/>
 		</transmission>
 		<transmission name="wrist_1_trans">
@@ -35,5 +35,5 @@
 				<mechanicalReduction>1</mechanicalReduction>
 			</actuator>
-			<joint name="${name}wrist_1_joint"/>
+			<joint name="${prefix}wrist_1_joint"/>
 		</transmission>
 		<transmission name="wrist_2_trans">
@@ -43,5 +43,5 @@
 				<mechanicalReduction>1</mechanicalReduction>
 			</actuator>
-			<joint name="${name}wrist_2_joint"/>
+			<joint name="${prefix}wrist_2_joint"/>
 		</transmission>
 		<transmission name="wrist_3_trans">
@@ -51,5 +51,5 @@
 				<mechanicalReduction>1</mechanicalReduction>
 			</actuator>
-			<joint name="${name}wrist_3_joint"/>
+			<joint name="${prefix}wrist_3_joint"/>
 		</transmission>
 	</xacro:macro>

File: ur_description/urdf/ur10.urdf.xacro (robot description, xacro)
@@ -4,5 +4,5 @@
        xmlns:interface="http://playerstage.sourceforge.net/gazebo/xmlschema/#interface"
        xmlns:xacro="http://ros.org/wiki/xacro">
-  <xacro:include filename="$(find ur_description)/urdf/ur10.transmission.xacro" />
+  <xacro:include filename="$(find ur_description)/urdf/ur.transmission.xacro" />
   <xacro:include filename="$(find ur_description)/urdf/ur10.gazebo.xacro" />
   <xacro:include filename="$(find ur_description)/urdf/materials.urdf.xacro" />
@@ -226,5 +226,5 @@
 		</inertial>
 	</link>
-  <xacro:ur10_arm_transmission prefix="${prefix}" />
+  <xacro:ur_arm_transmission prefix="${prefix}" />
   <xacro:ur10_arm_gazebo prefix="${prefix}" />
   </xacro:macro>

File: ur_description/urdf/ur10_robot.urdf.xacro (robot description, xacro)
@@ -5,6 +5,9 @@
        xmlns:xacro="http://playerstage.sourceforge.net/gazebo/xmlschema/#interface"
        name="ur10" >
-  <!-- common stuff -->
-  <xacro:include filename="$(find ur_description)/urdf/gazebo.urdf.xacro" />
+  <gazebo>
+    <plugin name="gazebo_ros_control" filename="libgazebo_ros_control.so">
+      <robotNamespace>/ur10</robotNamespace>
+    </plugin>
+  </gazebo>
   <!-- ur10 -->
   <xacro:include filename="$(find ur_description)/urdf/ur10.urdf.xacro" />

File: ur_description/urdf/ur5.urdf.xacro (robot description, xacro)
@@ -4,5 +4,5 @@
        xmlns:interface="http://playerstage.sourceforge.net/gazebo/xmlschema/#interface"
        xmlns:xacro="http://ros.org/wiki/xacro">
-  <xacro:include filename="$(find ur_description)/urdf/ur5.transmission.xacro" />
+  <xacro:include filename="$(find ur_description)/urdf/ur.transmission.xacro" />
   <xacro:include filename="$(find ur_description)/urdf/ur5.gazebo.xacro" />
   <xacro:include filename="$(find ur_description)/urdf/materials.urdf.xacro" />
@@ -229,5 +229,5 @@
   </joint>
   <link name="${prefix}ee_link" />
-  <xacro:ur5_arm_transmission name="${prefix}" />
+  <xacro:ur_arm_transmission prefix="${prefix}" />
   <gazebo reference="universal_robot">
     <material>Gazebo/Blue</material>

File: ur_description/urdf/ur5_robot.urdf.xacro (robot description, xacro)
@@ -5,6 +5,9 @@
        xmlns:xacro="http://playerstage.sourceforge.net/gazebo/xmlschema/#interface"
        name="ur5" >
-  <!-- common stuff -->
-  <xacro:include filename="$(find ur_description)/urdf/gazebo.urdf.xacro" />
+  <gazebo>
+    <plugin name="gazebo_ros_control" filename="libgazebo_ros_control.so">
+      <robotNamespace>/ur5</robotNamespace>
+    </plugin>
+  </gazebo>
   <!-- ur5 -->
   <xacro:include filename="$(find ur_description)/urdf/ur5.urdf.xacro" />
