Commit message: Update joint type to be continuous instead of revolute.

File: ur_description/urdf/ur10.urdf.xacro (robot description, xacro)
@@ -62,5 +62,5 @@
 		</inertial>
 	</link>
-	<joint name="${prefix}shoulder_pan_joint" type="revolute">
+	<joint name="${prefix}shoulder_pan_joint" type="continuous">
 		<parent link="${prefix}base_link" />
 		<child link = "${prefix}shoulder_link" />
@@ -88,5 +88,5 @@
 		</inertial>
 	</link>
-	<joint name="${prefix}shoulder_lift_joint" type="revolute">
+	<joint name="${prefix}shoulder_lift_joint" type="continuous">
 		<parent link="${prefix}shoulder_link" />
 		<child link = "${prefix}upper_arm_link" />
@@ -116,5 +116,5 @@
 		</inertial>
 	</link>
-	<joint name="${prefix}elbow_joint" type="revolute">
+	<joint name="${prefix}elbow_joint" type="continuous">
 		<parent link="${prefix}upper_arm_link" />
 		<child link = "${prefix}forearm_link" />
@@ -142,5 +142,5 @@
 		</inertial>
 	</link>
-	<joint name="${prefix}wrist_1_joint" type="revolute">
+	<joint name="${prefix}wrist_1_joint" type="continuous">
  		<parent link="${prefix}forearm_link" />
 		<child link = "${prefix}wrist_1_link" />
@@ -170,5 +170,5 @@
 		</inertial>
 	</link>
-	  <joint name="${prefix}wrist_2_joint" type="revolute">
+	  <joint name="${prefix}wrist_2_joint" type="continuous">
 		<parent link="${prefix}wrist_1_link" />
 		<child link = "${prefix}wrist_2_link" />
@@ -198,5 +198,5 @@
 		</inertial>
 	</link>
-	<joint name="${prefix}wrist_3_joint" type="revolute">
+	<joint name="${prefix}wrist_3_joint" type="continuous">
 		<parent link="${prefix}wrist_2_link" />
 		<child link = "${prefix}wrist_3_link" />

File: ur_description/urdf/ur5.urdf.xacro (robot description, xacro)
@@ -65,5 +65,5 @@
     </inertial>
   </link>
-  <joint name="${prefix}shoulder_pan_joint" type="revolute">
+  <joint name="${prefix}shoulder_pan_joint" type="continuous">
     <parent link="${prefix}base_link" />
     <child link = "${prefix}shoulder_link" />
@@ -91,5 +91,5 @@
     </inertial>
   </link>
-  <joint name="${prefix}shoulder_lift_joint" type="revolute">
+  <joint name="${prefix}shoulder_lift_joint" type="continuous">
     <parent link="${prefix}shoulder_link" />
     <child link = "${prefix}upper_arm_link" />
@@ -118,5 +118,5 @@
     </inertial>
   </link>
-  <joint name="${prefix}elbow_joint" type="revolute">
+  <joint name="${prefix}elbow_joint" type="continuous">
     <parent link="${prefix}upper_arm_link" />
     <child link = "${prefix}forearm_link" />
@@ -144,5 +144,5 @@
     </inertial>
   </link>
-  <joint name="${prefix}wrist_1_joint" type="revolute">
+  <joint name="${prefix}wrist_1_joint" type="continuous">
     <parent link="${prefix}forearm_link" />
     <child link = "${prefix}wrist_1_link" />
@@ -171,5 +171,5 @@
     </inertial>
   </link>
-  <joint name="${prefix}wrist_2_joint" type="revolute">
+  <joint name="${prefix}wrist_2_joint" type="continuous">
     <parent link="${prefix}wrist_1_link" />
     <child link = "${prefix}wrist_2_link" />
@@ -198,5 +198,5 @@
     </inertial>
   </link>
-  <joint name="${prefix}wrist_3_joint" type="revolute">
+  <joint name="${prefix}wrist_3_joint" type="continuous">
     <parent link="${prefix}wrist_2_link" />
     <child link = "${prefix}wrist_3_link" />
