Commit message: New controller parameters.

File: ur_description/urdf/ur5.urdf.xacro (robot description, xacro)
@@ -58,5 +58,5 @@
         <mesh filename="package://ur_description/meshes/ur5/collision/Base.dae" />
       </geometry>
-      <!-- <origin rpy="0.0 0.0 0.0" xyz="0.0 0.0 -0.009159"/> -->
+      <origin xyz="0.0 0.0 0.003" rpy="0.0 0.0 ${3.0 * pi / 4.0}" />
     </collision>
     <inertial>
@@ -83,5 +83,4 @@
         <mesh filename="package://ur_description/meshes/ur5/collision/Shoulder.dae" />
       </geometry>
-      <!-- <origin rpy="0.0 0.0 0.0" xyz="0.0 0.0 -0.009159"/> -->
     </collision>
     <inertial>
@@ -110,5 +109,5 @@
         <mesh filename="package://ur_description/meshes/ur5/collision/UpperArm.dae" />
       </geometry>
-<!--       <origin rpy="0.0 0.0 0.0" xyz="0.0 0.0 0.2125"/> -->
+      <origin xyz="0.0 0.0 0.0" rpy="0.0 0.0 0.0" />
     </collision>
     <inertial>
@@ -136,5 +135,4 @@
         <mesh filename="package://ur_description/meshes/ur5/collision/Forearm.dae" />
       </geometry>
-<!--       <origin rpy="0.0 0.0 0.0" xyz="0.0 0.0 0.196125"/> -->
     </collision>
     <inertial>
@@ -163,5 +161,5 @@
         <mesh filename="package://ur_description/meshes/ur5/collision/Wrist1.dae" />
       </geometry>
-      <origin rpy="0.0 1.570796325 0.0" xyz="0.0 0.093 0.0"/>
+      <origin xyz="0.0 ${wrist_1_length} 0.0" rpy="0.0 ${pi / 2.0} 0.0" />
     </collision>
     <inertial>
@@ -190,5 +188,5 @@
         <mesh filename="package://ur_description/meshes/ur5/collision/Wrist2.dae" />
       </geometry>
-       <origin rpy="0.0 0.0 0.0" xyz="0.0 0.0 0.09465"/>
+      <origin xyz="0.0 0.0 ${wrist_2_length}" rpy="0.0 0.0 0.0" />
     </collision>
     <inertial>
